Commit message: [add] added slideshow package and motor driver node

File: src/robot_arm/urdf/robot_arm.urdf (robot description, URDF)
Before this commit: robot gaze_arm, 10 links, 9 joints
Joints:
- joint joint3: limit lower=-0.5 upper=2.07 effort=0.5293 velocity=6.159937255 -> lower=-1.57 upper=1.57 effort=0.5293 velocity=6.159937255
- joint left_gripper_joint: limit lower=-0.5 upper=0.0 effort=1000.0 velocity=0.5 -> lower=0 upper=1.0 effort=1000.0 velocity=0.5; origin xyz=0 0.014 0.028 rpy=0 0 0 -> xyz=0 0.014 0.028 rpy=-1.0 0 0
- joint right_gripper_joint: limit (none) -> lower=0 upper=1.0 effort=1000.0 velocity=0.5; mimic (none) -> joint=left_gripper_joint multiplier=-1 offset=0; origin xyz=0 -0.014 0.028 rpy=0 0 0 -> xyz=0 -0.014 0.028 rpy=1.0 0 0; type fixed -> revolute

Commit message: [dev] coded robot_arm.launch

File: src/robot_arm/urdf/robot_arm.urdf (robot description, URDF)
Before this commit: robot robot_arm, 10 links, 9 joints
Joints:
- joint joint1: axis 0 1 0 -> 0 -1 0

Commit message: [add] added CAMERA.STL

File: src/robot_arm/urdf/robot_arm.urdf (robot description, URDF)
Before this commit: robot robot_arm, 10 links, 9 joints
Links:
- added link camera; visual mesh filename=package://robot_arm/urdf/CAMERA.STL scale=1 1 1
Joints:
- added joint camera_joint: type fixed, parent gripper_base, child camera, origin xyz=-0.035 0.018 0.058 rpy=0 0 0
